Commit message: second commit

File: assets/submarine.urdf (robot description, URDF)
Before this commit: robot submarine, 15 links, 14 joints
Links:
- removed link base_link
Joints:
- removed joint body_link
- joint Main_motor_joint: axis 0 1 0 -> (none); limit effort=2000.0 velocity=100.0 -> (none); type continuous -> fixed
- joint Motor_down1_joint: axis 0 0 1 -> (none); limit effort=500.0 velocity=100.0 -> (none); type continuous -> fixed
- joint Motor_down2_joint: axis 0 0 1 -> (none); limit effort=500.0 velocity=100.0 -> (none); type continuous -> fixed
- joint Motor_left1_joint: axis 1 0 0 -> (none); limit effort=500.0 velocity=100.0 -> (none); type continuous -> fixed
- joint Motor_left2_joint: axis 1 0 0 -> (none); limit effort=500.0 velocity=100.0 -> (none); type continuous -> fixed
- joint Motor_left_joint: axis 0 0 1 -> (none); limit effort=500.0 velocity=100.0 -> (none); type continuous -> fixed
- joint Motor_right1_joint: axis 1 0 0 -> (none); limit effort=500.0 velocity=100.0 -> (none); type continuous -> fixed
- joint Motor_right2_joint: axis 1 0 0 -> (none); limit effort=500.0 velocity=100.0 -> (none); type continuous -> fixed
- joint Motor_right_joint: axis 0 0 1 -> (none); limit effort=500.0 velocity=100.0 -> (none); type continuous -> fixed
- joint Motor_up1_joint: axis 0 0 1 -> (none); limit effort=500.0 velocity=100.0 -> (none); type continuous -> fixed
- joint Motor_up2_joint: axis 0 0 1 -> (none); limit effort=500.0 velocity=100.0 -> (none); type continuous -> fixed

Commit message: third commit

File: assets/submarine.urdf (robot description, URDF)
Before this commit: robot submarine, 14 links, 13 joints
Links:
- link Main_motor_link: mass 13.264 -> 0.01
- link Motor_down1_link: mass 0.7525 -> 0.01
- link Motor_down2_link: mass 0.7525 -> 0.01
- link Motor_left1_link: mass 0.7525 -> 0.01
- link Motor_left2_link: mass 0.7525 -> 0.01
- link Motor_left_link: mass 0.2348439 -> 0.01
- link Motor_right1_link: mass 0.7525 -> 0.01
- link Motor_right2_link: mass 0.7525 -> 0.01
- link Motor_right_link: mass 0.2348439 -> 0.01
- link Motor_up1_link: mass 0.7525 -> 0.01
- link Motor_up2_link: mass 0.7525 -> 0.01
